File: solenoid_board.sch (KiCad schematic (older format))
At the start: 48 parts, among them J2 MCU_LEFT_LEGS, J3 MCU_RIGHT_LEGS

Commit message: Finished laying out Scoreboard PCB, good enough for government work.
Connections:
- net D10: now also Driver1.1 (Pin_1); no longer Driver1.7 (Pin_7)
- net D5: now also Driver1.7 (Pin_7); no longer Driver1.6 (Pin_6)
- net D6: now also Driver1.6 (Pin_6); no longer Driver1.2 (Pin_2)
- net D9: now also Driver1.2 (Pin_2); no longer Driver1.1 (Pin_1)
- removed net dp: 7Seg_1.5 (Pin_5), 7Seg_2.5 (Pin_5), 7Seg_3.5 (Pin_5), 7Seg_4.5 (Pin_5), 7Seg_5.5 (Pin_5), 7Seg_6.5 (Pin_5), 7Seg_7.5 (Pin_5), 7Seg_8.5 (Pin_5)
- no-connect marks 4 -> 12
Changed lines of the file:
@@
 Text Label 2550 5000 0    50   ~ 0
 g
-Text Label 2050 5000 2    50   ~ 0
-dp
 $Comp
 L Connector_Generic:Conn_01x02 +5VIN1
@@
 Text Label 2550 5750 0    50   ~ 0
 g
-Text Label 2050 5750 2    50   ~ 0
-dp
 $Comp
 L Connector_Generic:Conn_02x05_Top_Bottom 7Seg_2
@@
 Text Label 2550 6600 0    50   ~ 0
 g
-Text Label 2050 6600 2    50   ~ 0
-dp
 $Comp
 L Connector_Generic:Conn_02x05_Top_Bottom 7Seg_3
@@
 Text Label 2550 7400 0    50   ~ 0
 g
-Text Label 2050 7400 2    50   ~ 0
-dp
 $Comp
 L Connector_Generic:Conn_02x05_Top_Bottom 7Seg_4
@@
 	5650 1550 5050 1550
 Text Label 7650 1000 2    50   ~ 0
+D10
+Text Label 7650 1100 2    50   ~ 0
 D9
-Text Label 7650 1100 2    50   ~ 0
+Text Label 7650 1500 2    50   ~ 0
 D6
-Text Label 7650 1500 2    50   ~ 0
+Text Label 7650 1600 2    50   ~ 0
 D5
-Text Label 7650 1600 2    50   ~ 0
-D10
 Text Label 7650 1200 2    50   ~ 0
 LT
@@
 Text Label 4750 5050 0    50   ~ 0
 g
-Text Label 4250 5050 2    50   ~ 0
-dp
 $Comp
 L Connector_Generic:Conn_02x05_Top_Bottom 7Seg_5
@@
 Text Label 4750 5800 0    50   ~ 0
 g
-Text Label 4250 5800 2    50   ~ 0
-dp
 $Comp
 L Connector_Generic:Conn_02x05_Top_Bottom 7Seg_6
@@
 Text Label 4750 6650 0    50   ~ 0
 g
-Text Label 4250 6650 2    50   ~ 0
-dp
 $Comp
 L Connector_Generic:Conn_02x05_Top_Bottom 7Seg_7
@@
 Text Label 4750 7450 0    50   ~ 0
 g
-Text Label 4250 7450 2    50   ~ 0
-dp
 $Comp
 L Connector_Generic:Conn_02x05_Top_Bottom 7Seg_8
@@
 	8650 1300 8650 1400
 $Comp
-L power:GND #PWR?
+L power:GND #PWR0111
 U 1 1 5E98C6F5
 P 8650 1400
-F 0 "#PWR?" H 8650 1150 50  0001 C CNN
+F 0 "#PWR0111" H 8650 1150 50  0001 C CNN
 F 1 "GND" H 8655 1227 50  0000 C CNN
 F 2 "" H 8650 1400 50  0001 C CNN
@@
 	8150 1000 8650 1000
 Connection ~ 8650 1000
+NoConn ~ 4250 5050
+NoConn ~ 2050 5000
+NoConn ~ 2050 5750
+NoConn ~ 2050 6600
+NoConn ~ 2050 7400
+NoConn ~ 4250 7450
+NoConn ~ 4250 6650
+NoConn ~ 4250 5800
 $EndSCHEMATC
